Commit message: Update PRS_Robot.urdf

File: robot/PRS_Robot.urdf (robot description, URDF)
Before this commit: robot Xbot, 7 links, 6 joints
Joints:
- joint joint_base: limit lower=-0.5 upper=0.5 effort=30 velocity=1.0 -> lower=-0.8 upper=0.8 effort=30 velocity=1.0
- joint joint_big: limit lower=-0.5 upper=1 effort=30 velocity=1.7 -> lower=-0.5 upper=1.5 effort=30 velocity=1.7
- joint joint_hand: limit lower=-1.6 upper=1.0 effort=30 velocity=1.6 -> lower=-1.6 upper=1.6 effort=30 velocity=1.6
- joint joint_small: limit lower=-0.0 upper=1 effort=30 velocity=2.0 -> lower=-0.0 upper=2 effort=30 velocity=2.0

Commit message: Update PRS_Robot.urdf

File: robot/PRS_Robot.urdf (robot description, URDF)
Before this commit: robot Xbot, 7 links, 6 joints
Joints:
- joint joint_base: limit lower=-0.8 upper=0.8 effort=30 velocity=1.0 -> lower=-0.6 upper=0.6 effort=30 velocity=1.0
- joint joint_big: limit lower=-0.5 upper=1.5 effort=30 velocity=1.7 -> lower=-0.5 upper=1.4 effort=30 velocity=1.7
- joint joint_small: limit lower=-0.0 upper=2 effort=30 velocity=2.0 -> lower=-0.0 upper=1.7 effort=30 velocity=2.0

Commit message: Update PRS_Robot.urdf

File: robot/PRS_Robot.urdf (robot description, URDF)
Before this commit: robot Xbot, 7 links, 6 joints
Joints:
- joint joint_base: limit lower=-0.6 upper=0.6 effort=30 velocity=1.0 -> lower=-0.5 upper=0.5 effort=30 velocity=1.0
